Commit message: Generalizing urdf paths, adding rviz

File: urdf/rover_5.urdf (robot description, URDF)
Before this commit: robot rover_5, 9 links, 8 joints
Links:
- link base_link: geometry visual mesh filename=file:///$(arg meshDirectory)/base_link.stl
- link intel_realsense: geometry visual mesh filename=file:///$(arg meshDirectory)/Intel_RealSense_Depth_Camera_D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 scale=.001 .001 .001
- link top_rack: geometry visual mesh filename=file:///$(arg meshDirectory)/rack.stl
- link wheel_1: geometry visual mesh filename=file:///$(arg meshDirectory)/wheel_scaled.stl
- link wheel_2: geometry visual mesh filename=file:///$(arg meshDirectory)/wheel_scaled.stl
- link wheel_3: geometry visual mesh filename=file:///$(arg meshDirectory)/wheel_scaled.stl
- link wheel_4: geometry visual mesh filename=file:///$(arg meshDirectory)/wheel_scaled.stl

Commit message: Mapping is...working, to a degree. Pathplanning is next on the docket

File: urdf/rover_5.urdf (robot description, URDF)
Before this commit: robot rover_5, 9 links, 8 joints
Links:
- removed link phidgets_imu
- added link imu; visual box size=.038 .014 .038
Joints:
- removed joint base_to_phidgets
- added joint base_to_imu: type fixed, parent base_link, child imu, origin xyz=-.265 .1 .04

Commit message: Bug bash, fixed joy_node param issue

File: urdf/rover_5.urdf (robot description, URDF)
Before this commit: robot rover_5, 9 links, 8 joints
Links:
- removed link imu
- added link imu_link; visual box size=.038 .014 .038
Joints:
- removed joint base_to_imu
- added joint base_to_imu_link: type fixed, parent base_link, child imu_link, origin xyz=-.265 .1 .04

Commit message: Mounting of IMU vs TF representation can be important.

File: urdf/rover_5.urdf (robot description, URDF)
Before this commit: robot rover_5, 9 links, 8 joints
Links:
- link imu_link: geometry visual box size=.038 .038 .014
Joints:
- joint base_to_imu_link: origin xyz=-.265 .1 .04 -> xyz=-.265 .1 .04 rpy=0 0 0

Commit message: Unfucked meshes and URDF

File: urdf/rover_5.urdf (robot description, URDF)
Before this commit: robot rover_5, 9 links, 8 joints
Links:
- removed link imu_link
- removed link usb_gps
- link base_link: geometry visual mesh filename=file:///$(arg meshDirectory)/base_link_scaled.stl
Joints:
- removed joint base_to_imu_link
- removed joint rack_to_gps
- joint base_to_rack: origin xyz=-.353 .0944 .058 -> xyz=-.085 .05 .044
- joint base_to_wheel_1: origin xyz=-.3542 0 0 -> xyz=-.088 -.095 -.014
- joint base_to_wheel_2: origin xyz=-.18 0 0 -> xyz=.088 -.095 -.014
- joint base_to_wheel_3: origin xyz=-.3542 .09 0 -> xyz=.088 .095 -.014
- joint base_to_wheel_4: origin xyz=-.18 .09 0 -> xyz=-.088 .095 -.014
